Commit message: update robot model

File: src/hyper_robot2/urdf/hyper_robot2.urdf (robot description, URDF)
Before this commit: robot hyper_robot, 7 links, 6 joints
Links:
- link Link1: mass 0.11358 -> 0.11138; geometry collision mesh filename=package://hyper_robot2/meshes/Link1.STL; visual mesh filename=package://hyper_robot2/meshes/Link1.STL
- link Link2: geometry collision mesh filename=package://hyper_robot2/meshes/Link2.STL; visual mesh filename=package://hyper_robot2/meshes/Link2.STL
- link Link3: geometry collision mesh filename=package://hyper_robot2/meshes/Link3.STL; visual mesh filename=package://hyper_robot2/meshes/Link3.STL
- link Link4: geometry collision mesh filename=package://hyper_robot2/meshes/Link4.STL; visual mesh filename=package://hyper_robot2/meshes/Link4.STL
- link Link5: geometry collision mesh filename=package://hyper_robot2/meshes/Link5.STL; visual mesh filename=package://hyper_robot2/meshes/Link5.STL
- link Link6: geometry collision mesh filename=package://hyper_robot2/meshes/Link6.STL; visual mesh filename=package://hyper_robot2/meshes/Link6.STL
- link base_link: geometry collision mesh filename=package://hyper_robot2/meshes/base_link.STL; visual mesh filename=package://hyper_robot2/meshes/base_link.STL
Joints:
- joint Joint0: limit lower=-3.14 upper=3.14 effort=1 velocity=1 -> (none); origin xyz=-0.02 0 0 rpy=-3.1416 0 -0.00 -> xyz=0.02 0 -0.07755 rpy=0 0 0
- joint Joint1: limit lower=-3.14 upper=3.14 effort=1 velocity=1 -> (none); origin xyz=-0.0465 0 0.08365 rpy=1.5708 -0 0 -> xyz=0.0465 0 -0.1031 rpy=-1.5708 0 3.1416
- joint Joint2: limit lower=-3.14 upper=3.14 effort=1 velocity=1 -> (none); origin xyz=0.0 0.06364 -0.0 rpy=-0.00 0 0.0 -> xyz=0 0.06365 0 rpy=0 0 0
- joint Joint3: limit lower=-3.14 upper=3.14 effort=1 velocity=1 -> (none); origin xyz=0.027199 0.025358 0.00080668 rpy=1.5714 1.5714 0.0 -> xyz=0.02565 0.031 0 rpy=-1.5708 -1.5708 0
- joint Joint4: limit lower=-3.14 upper=3.14 effort=1 velocity=1 -> (none); origin xyz=0 0 -0.1062 rpy=-1.5708 0.0 -3.1416 -> xyz=0 0 0.09265 rpy=1.5708 0 0
- joint Joint5: limit lower=-3.14 upper=3.14 effort=1 velocity=1 -> (none); origin xyz=0 0.031993 -0.03165 rpy=-1.5714 0 0 -> xyz=0 0.031 -0.04165 rpy=-1.5708 0 0
