Commit message: add rotation freedom to MarkPen by adding additional joint

File: src/hyper_robot3/urdf/hyper_robot3.urdf (robot description, URDF)
Before this commit: robot hyper_robot3, 8 links, 7 joints
Links:
- added link MarkPen, mass 0.012663; collision mesh filename=package://hyper_robot3/meshes/MarkPen.STL; visual mesh filename=package://hyper_robot3/meshes/MarkPen.STL
- added link free_endeffector
- added link freedom_roll
- link Link5: mass 0.0928720201733155 -> 0.092872
- link Link6: mass 0.0160210321477213 -> 0.016021
- link base_link: mass 1.40368130340825 -> 1.40368124385494
- link end_effector: mass 0.015815 -> 0.0031515
Joints:
- added joint JointPen: type revolute, parent end_effector, child MarkPen, origin xyz=0 0 0 rpy=1.5708 0 2.433, axis 0 1 0, limit lower=-1.5708 upper=1.5708 effort=1 velocity=1
- added joint JointPenPitch: type revolute, parent freedom_roll, child free_endeffector, axis 0 0 1, limit lower=-1.5708 upper=1.5708 effort=1 velocity=1
- added joint JointPenRoll: type revolute, parent MarkPen, child freedom_roll, axis 1 0 0, limit lower=-1.5708 upper=1.5708 effort=1 velocity=1
- joint Joint0: limit (none) -> lower=-1.5707 upper=1.5707 effort=1 velocity=1; origin xyz=0.0200000000000002 0 -0.18065 rpy=0 0 0 -> xyz=0.02 0 -0.18065 rpy=0 0 0; type continuous -> revolute
- joint Joint1: limit (none) -> lower=-1.5707 upper=1.5707 effort=1 velocity=1; origin xyz=0.0464999999999984 0 0 rpy=1.57079632679491 1.5707963267949 0 -> xyz=0.0465 0 0 rpy=1.5708 1.5708 0; type continuous -> revolute
- joint Joint2: axis 0 0 0.999999999996974 -> 0 0 1; limit (none) -> lower=-1.5707 upper=1.5707 effort=1 velocity=1; origin xyz=0.06365 0 0 rpy=0 0 -1.5707963267949 -> xyz=0.06365 0 0 rpy=0 0 -1.5708; type continuous -> revolute
- joint Joint3: limit (none) -> lower=-1.5707 upper=1.5707 effort=1 velocity=1; origin xyz=0.0256499999999205 0.12365 0 rpy=-1.57079632679475 0 0 -> xyz=0.02565 0.12365 0 rpy=-1.5708 0 0; type continuous -> revolute
- joint Joint4: limit (none) -> lower=-1.5707 upper=1.5707 effort=1 velocity=1; origin xyz=0.0416500000000051 0 0 rpy=1.57079632679479 0 -1.5707963267949 -> xyz=0.04165 0 0 rpy=1.5708 0 -1.5708; type continuous -> revolute
- joint Joint5: limit (none) -> lower=-1.5707 upper=1.5707 effort=1 velocity=1; origin xyz=0 0 0 rpy=-1.57079632679479 0 0 -> xyz=0 0 0 rpy=-1.5708 0 0; type continuous -> revolute
- joint JointEnd: limit (none) -> lower=-1.5707 upper=1.5707 effort=1 velocity=1

Commit message: gazebo_robot,hyper_control,hyper_robot5

File: src/hyper_robot3/urdf/hyper_robot3.urdf (robot description, URDF)
Before this commit: robot hyper_robot3, 11 links, 10 joints
Joints:
- joint Joint0: limit lower=-1.5707 upper=1.5707 effort=1 velocity=1 -> lower=-2.3561 upper=2.3561 effort=10 velocity=1
- joint JointPen: limit lower=-1.5708 upper=1.5708 effort=1 velocity=1 -> lower=-3.142857 upper=3.142857 effort=1 velocity=1; origin xyz=0 0 0 rpy=1.5708 0 2.433 -> xyz=0 0 0 rpy=1.5708 0 0
- joint JointPenPitch: limit lower=-1.5708 upper=1.5708 effort=1 velocity=1 -> lower=-0.7854 upper=0.7854 effort=1 velocity=1
- joint JointPenRoll: limit lower=-1.5708 upper=1.5708 effort=1 velocity=1 -> lower=-0.7854 upper=0.7854 effort=1 velocity=1
