Commit message: link gazebo_robot to px4

File: src/gazebo_robot/model/hyper_robot4/hyper_robot4.xacro.urdf (robot description, URDF)
Before this commit: robot hyper_robot4, 13 links, 12 joints
Links:
- added link /imu_link, mass 0.015
Joints:
- added joint /imu_joint: type revolute, parent base_link, child /imu_link, origin xyz=0 0 0 rpy=0 0 0, axis 0 0 1, limit lower=0 upper=0 effort=0 velocity=0

Commit message: setup px4 command and robot control in gazebo

File: src/gazebo_robot/model/hyper_robot4/hyper_robot4.xacro.urdf (robot description, URDF)
Before this commit: robot hyper_robot4, 14 links, 13 joints
Links:
- link base_link: mass 1.4037 -> 1.4; geometry collision box size=0.4 0.4 0.2; visual mesh filename=package://hyper_robot4/meshes/base_link.STL
Joints:
- joint rotor_0_joint: axis 0 1 0 -> 0 0 1; origin xyz=0.15778 -0.15778 0.022914 rpy=-1.5708 0 1.7863 -> xyz=0.15778 -0.15778 0.022914 rpy=0 0 0
- joint rotor_1_joint: axis 0 1 0 -> 0 0 1; origin xyz=-0.15778 0.15778 0.022914 rpy=-1.5708 0 1.7179 -> xyz=-0.15778 0.15778 0.022914 rpy=0 0 0
- joint rotor_2_joint: axis 0 1 0 -> 0 0 1; origin xyz=0.15778 0.15778 0.0245 rpy=1.5708 0 0.18169 -> xyz=0.15778 0.15778 0.0245 rpy=0 0 0
- joint rotor_3_joint: axis 0 1 0 -> 0 0 1; origin xyz=-0.15778 -0.15778 0.02285 rpy=-1.5708 0 -2.9802 -> xyz=-0.15778 -0.15778 0.02285 rpy=0 0 0

Commit message: update xacro,but some control problem exist:imu accelemeter not stable

File: src/gazebo_robot/model/hyper_robot4/hyper_robot4.xacro.urdf (robot description, URDF)
Before this commit: robot hyper_robot4, 14 links, 13 joints
Links:
- added link imu_middle
- link /imu_link: geometry visual box size=0.01 0.01 0.01
Joints:
- added joint /imu_prismatic: type prismatic, parent base_link, child imu_middle, origin xyz=0 0 0 rpy=0 0 0, axis 0 0 1, limit lower=-0.01 upper=0.01 effort=0 velocity=0
- joint /imu_joint: origin xyz=0 0 0 rpy=0 0 0 -> xyz=0 0 0.02 rpy=0 0 0
